Commit message: Move dashboard to src/robie_safety/web; accept /sw/estop in safety_node

File: src/robie_bringup/urdf/robie.urdf (robot description, URDF)
Before this commit: robot robie, 2 links, 1 joints
Links:
- removed link base_scan
- added link base_plate; visual box size=0.42 0.32 0.01
- added link front_left_wheel; visual cylinder length=0.04 radius=0.05
- added link front_right_wheel; visual cylinder length=0.04 radius=0.05
- added link lidar_link; visual cylinder length=0.06 radius=0.04
- added link rear_left_wheel; visual cylinder length=0.04 radius=0.05
- added link rear_right_wheel; visual cylinder length=0.04 radius=0.05
- added link top_plate; visual box size=0.38 0.28 0.02
- link base_link: mass 10 -> 8.0; geometry collision box size=0.40 0.30 0.15; visual box size=0.40 0.30 0.15
Joints:
- removed joint scan_joint
- added joint base_plate_joint: type fixed, parent base_link, child base_plate, origin xyz=0 0 -0.01 rpy=0 0 0
- added joint front_left_wheel_joint: type continuous, parent base_link, child front_left_wheel, origin xyz=0.15 0.15 0.0 rpy=0 0 0, axis 0 1 0
- added joint front_right_wheel_joint: type continuous, parent base_link, child front_right_wheel, origin xyz=0.15 -0.15 0.0 rpy=0 0 0, axis 0 1 0
- added joint lidar_joint: type fixed, parent top_plate, child lidar_link, origin xyz=0.05 0 0.02 rpy=0 0 0
- added joint rear_left_wheel_joint: type continuous, parent base_link, child rear_left_wheel, origin xyz=-0.15 0.15 0.0 rpy=0 0 0, axis 0 1 0
- added joint rear_right_wheel_joint: type continuous, parent base_link, child rear_right_wheel, origin xyz=-0.15 -0.15 0.0 rpy=0 0 0, axis 0 1 0
- added joint top_plate_joint: type fixed, parent base_link, child top_plate, origin xyz=0 0 0.15 rpy=0 0 0
